Commit message: fix: update URDF file paths

File: ros2_ws/src/robot_description/urdf/HARP2_urdf/arm/arm.urdf.xacro (robot description, xacro)
@@ -3,6 +3,12 @@
     xmlns:xacro="http://ros.org/wiki/xacro">
     <xacro:include filename="$(find robot_description)/urdf/meshes/standard_inertia_util.xacro" />
+    <xacro:macro name="harp2_arm" params="parent_link:=base_link prefix:=arm_ xyz:='0 0 0.26' rpy:='0 0 0' visual_only:=true">
+    <joint name="${prefix}mount_joint" type="fixed">
+        <parent link="${parent_link}"/>
+        <child link="${prefix}base_link"/>
+        <origin xyz="${xyz}" rpy="${rpy}"/>
+    </joint>
     <!-- Base -->
-    <link name="base_link">
+    <link name="${prefix}base_link">
         <visual>
             <origin xyz="0 0 0" rpy="0 0 0"/>
@@ -11,19 +17,23 @@
             </geometry>
         </visual>
-        <collision>
-            <origin xyz="0 0 0" rpy="0 0 0"/>
-            <geometry>
-                <mesh filename="file://$(find robot_description)/urdf/HARP2_urdf/arm/meshes/arm_baselink.dae"/>
-            </geometry>
-        </collision>
+        <xacro:unless value="${visual_only}">
+            <collision>
+                <origin xyz="0 0 0" rpy="0 0 0"/>
+                <geometry>
+                    <mesh filename="file://$(find robot_description)/urdf/HARP2_urdf/arm/meshes/arm_baselink.dae"/>
+                </geometry>
+            </collision>
+        </xacro:unless>
     </link>
-    <joint name="prismatic_joint" type="prismatic">
-        <parent link="base_link"/>
-        <child link="Lx16a_1"/>
+    <joint name="${prefix}prismatic_joint" type="${'fixed' if visual_only else 'prismatic'}">
+        <parent link="${prefix}base_link"/>
+        <child link="${prefix}Lx16a_1"/>
         <origin xyz="0 -0.04070000 0" rpy="0 0 0"/>
-        <axis xyz="0 0 1"/>
-        <limit lower="-0.105" upper="0.095" effort="100.0" velocity="0.5"/>
+        <xacro:unless value="${visual_only}">
+            <axis xyz="0 0 1"/>
+            <limit lower="-0.105" upper="0.095" effort="100.0" velocity="0.5"/>
+        </xacro:unless>
     </joint>
-    <link name="Lx16a_1">
+    <link name="${prefix}Lx16a_1">
         <visual>
             <origin xyz="0 0.04070000 0" rpy="0 0 0"/>
@@ -32,23 +42,27 @@
             </geometry>
         </visual>
-        <collision>
-            <origin xyz="0 0.04070000 0" rpy="0 0 0"/>
-            <geometry>
-                <mesh filename="file://$(find robot_description)/urdf/HARP2_urdf/arm/meshes/Lx16a_1.dae"/>
-            </geometry>
-        </collision>
-        <xacro:inertial_box mass="0.06" x="0.0245" y="0.0507" z="0.035">
-				<origin xyz="0 0.01474695 0" rpy="0 0 0"/>
-		</xacro:inertial_box>
+        <xacro:unless value="${visual_only}">
+            <collision>
+                <origin xyz="0 0.04070000 0" rpy="0 0 0"/>
+                <geometry>
+                    <mesh filename="file://$(find robot_description)/urdf/HARP2_urdf/arm/meshes/Lx16a_1.dae"/>
+                </geometry>
+            </collision>
+            <xacro:inertial_box mass="0.06" x="0.0245" y="0.0507" z="0.035">
+				    <origin xyz="0 0.01474695 0" rpy="0 0 0"/>
+		    </xacro:inertial_box>
+        </xacro:unless>
     </link>
-    <joint name="joint_1" type="revolute">
+    <joint name="${prefix}joint_1" type="${'fixed' if visual_only else 'revolute'}">
         <origin xyz="0 0 -0.03383600" rpy="3.14159 0 -1.0472"/>
-        <parent link="Lx16a_1"/>
-        <child link="Lx16a_2"/>
-        <axis xyz="0 0 1"/>
-        <limit lower="0" upper="4.1887902" effort="10.0" velocity="1.0"/>
-        <joint_properties friction="0.0"/>
+        <parent link="${prefix}Lx16a_1"/>
+        <child link="${prefix}Lx16a_2"/>
+        <xacro:unless value="${visual_only}">
+            <axis xyz="0 0 1"/>
+            <limit lower="0" upper="4.1887902" effort="10.0" velocity="1.0"/>
+            <joint_properties friction="0.0"/>
+        </xacro:unless>
     </joint>
-    <link name="Lx16a_2">
+    <link name="${prefix}Lx16a_2">
         <visual>
             <origin xyz="0 0.04070000 0.03383600" rpy="0 0 0"/>
@@ -57,23 +71,27 @@
             </geometry>
         </visual>
-        <collision>
-            <origin xyz="0 0.04070000 0.03383600" rpy="0 0 0"/>
-            <geometry>
-                <mesh filename="file://$(find robot_description)/urdf/HARP2_urdf/arm/meshes/Lx16a_2.dae"/>
-            </geometry>
-        </collision>
-        <xacro:inertial_box mass="0.06" x="0.0245" y="0.0492" z="0.035">
-				<origin xyz="0 0.01174695 0" rpy="0 0 0"/>
-		</xacro:inertial_box>
+        <xacro:unless value="${visual_only}">
+            <collision>
+                <origin xyz="0 0.04070000 0.03383600" rpy="0 0 0"/>
+                <geometry>
+                    <mesh filename="file://$(find robot_description)/urdf/HARP2_urdf/arm/meshes/Lx16a_2.dae"/>
+                </geometry>
+            </collision>
+            <xacro:inertial_box mass="0.06" x="0.0245" y="0.0492" z="0.035">
+				    <origin xyz="0 0.01174695 0" rpy="0 0 0"/>
+		    </xacro:inertial_box>
+        </xacro:unless>
     </link>
-    <joint name="joint_2" type="revolute">
+    <joint name="${prefix}joint_2" type="${'fixed' if visual_only else 'revolute'}">
         <origin xyz="0 0 0" rpy="-2.0943951 0 3.14159265"/>
-        <parent link="Lx16a_2"/>
-        <child link="wrist2end_effector"/>
-        <axis xyz="1 0 0"/>
-        <limit lower="0" upper="4.1887902" effort="10.0" velocity="1.0"/>
-        <joint_properties friction="0.0"/>
+        <parent link="${prefix}Lx16a_2"/>
+        <child link="${prefix}wrist2end_effector"/>
+        <xacro:unless value="${visual_only}">
+            <axis xyz="1 0 0"/>
+            <limit lower="0" upper="4.1887902" effort="10.0" velocity="1.0"/>
+            <joint_properties friction="0.0"/>
+        </xacro:unless>
     </joint>
-    <link name="wrist2end_effector">
+    <link name="${prefix}wrist2end_effector">
         <visual>
             <origin xyz="0 0 0" rpy="0 0 0"/>
@@ -82,20 +100,22 @@
             </geometry>
         </visual>
-        <collision>
-            <origin xyz="0 0 0" rpy="0 0 0"/>
-            <geometry>
-                <mesh filename="file://$(find robot_description)/urdf/HARP2_urdf/arm/meshes/wrist2end_effector.dae"/>
-            </geometry>
-        </collision>
-        <xacro:inertial_box mass="0.004" x="0.044" y="0.02800297" z="0.022">
-				<origin xyz="0.0005 0.009982745 0" rpy="0 0 0"/>
-		</xacro:inertial_box>
+        <xacro:unless value="${visual_only}">
+            <collision>
+                <origin xyz="0 0 0" rpy="0 0 0"/>
+                <geometry>
+                    <mesh filename="file://$(find robot_description)/urdf/HARP2_urdf/arm/meshes/wrist2end_effector.dae"/>
+                </geometry>
+            </collision>
+            <xacro:inertial_box mass="0.004" x="0.044" y="0.02800297" z="0.022">
+				    <origin xyz="0.0005 0.009982745 0" rpy="0 0 0"/>
+		    </xacro:inertial_box>
+        </xacro:unless>
     </link>
-    <joint name="fixed_joint" type="fixed">
-        <parent link="wrist2end_effector"/>
-        <child link="end_effector"/>
+    <joint name="${prefix}fixed_joint" type="fixed">
+        <parent link="${prefix}wrist2end_effector"/>
+        <child link="${prefix}end_effector"/>
         <origin xyz="0 0 0" rpy="0 0 0"/>
     </joint>
-    <link name="end_effector">
+    <link name="${prefix}end_effector">
         <visual>
             <origin xyz="0 0 0" rpy="0 3.14159 0"/>
@@ -104,13 +124,16 @@
             </geometry>
         </visual>
-        <collision>
-            <origin xyz="0 0 0" rpy="0 3.14159 0"/>
-            <geometry>
-                <mesh filename="file://$(find robot_description)/urdf/HARP2_urdf/arm/meshes/end_effector.dae"/>
-            </geometry>
-        </collision>
-        <xacro:inertial_box mass="0.065" x="0.07248686" y="0.05971815" z="0.084">
-				<origin xyz="0 0.058859075 -0.009" rpy="0 0 0"/>
-		</xacro:inertial_box>
+        <xacro:unless value="${visual_only}">
+            <collision>
+                <origin xyz="0 0 0" rpy="0 3.14159 0"/>
+                <geometry>
+                    <mesh filename="file://$(find robot_description)/urdf/HARP2_urdf/arm/meshes/end_effector.dae"/>
+                </geometry>
+            </collision>
+            <xacro:inertial_box mass="0.065" x="0.07248686" y="0.05971815" z="0.084">
+				    <origin xyz="0 0.058859075 -0.009" rpy="0 0 0"/>
+		    </xacro:inertial_box>
+        </xacro:unless>
     </link>
+    </xacro:macro>
 </robot>

File: ros2_ws/src/robot_description/urdf/HARP2_urdf/robot.urdf.xacro (robot description, xacro)
@@ -4,6 +4,10 @@
     <xacro:include filename="$(find robot_description)/urdf/meshes/standard_inertia_util.xacro" />
     <xacro:include filename="$(find robot_description)/urdf/HARP2_urdf/holonomic_wheel/wheel.xacro" />
+    <xacro:include filename="$(find robot_description)/urdf/HARP2_urdf/arm/arm.urdf.xacro" />
+    <xacro:include filename="$(find robot_description)/urdf/imu/imu.xacro" />
+    <xacro:include filename="$(find robot_description)/urdf/paa5160/paa5160.xacro" />
     <xacro:arg name="use_TopicBasedSystem_hardware_interface" default="false"/>
     <xacro:arg name="use_controller" default="false"/>
+    <xacro:arg name="enable_gazebo_imu" default="false"/>
     <!-- Hhardware interfaces chosen according to whether the robot is simulated or real -->
     <xacro:if value="$(arg use_controller)">
@@ -73,3 +77,5 @@
     <!-- Add YDlidar_X4 -->
     <xacro:include filename="$(find robot_description)/urdf/HARP2_urdf/lidar/YDlidar_X4/lidar.xacro" />
+    <!-- Add auxiliary sensors and arm -->
+    <xacro:harp2_arm parent_link="base_link" prefix="arm_" xyz="0 0 0.26" rpy="0 0 0"/>
 </robot>
